Commit message: added state estimation package + imu plugins

File: examples/fws_robot_harmonic/src/fws_robot_description/gazebo/fws_robot.gazebo.xacro (robot description, xacro)
@@ -10,4 +10,26 @@
         <render_engine>ogre2</render_engine>
       </plugin>
+      <plugin filename="gz-sim-imu-system" name="gz::sim::systems::Imu"/>
+    </gazebo>
+    <gazebo reference="imu_link">
+      <sensor name="imu_sensor" type="imu">
+        <gz_frame_id>imu_link</gz_frame_id>
+        <topic>imu</topic>
+        <update_rate>100</update_rate>
+        <imu>
+          <angular_velocity>
+            <x><noise type="gaussian"><mean>0</mean><stddev>2e-4</stddev></noise></x>
+            <y><noise type="gaussian"><mean>0</mean><stddev>2e-4</stddev></noise></y>
+            <z><noise type="gaussian"><mean>0</mean><stddev>2e-4</stddev></noise></z>
+          </angular_velocity>
+          <linear_acceleration>
+            <x><noise type="gaussian"><mean>0</mean><stddev>1.7e-2</stddev></noise></x>
+            <y><noise type="gaussian"><mean>0</mean><stddev>1.7e-2</stddev></noise></y>
+            <z><noise type="gaussian"><mean>0</mean><stddev>1.7e-2</stddev></noise></z>
+          </linear_acceleration>
+        </imu>
+        <alwaysOn>true</alwaysOn>
+        <visualize>false</visualize>
+      </sensor>
     </gazebo>
     <gazebo reference="lidar_head_link" >

File: examples/fws_robot_harmonic/src/fws_robot_description/robots/fws_robot.urdf.xacro (robot description, xacro)
@@ -9,4 +9,5 @@
   <xacro:include filename="$(find fws_robot_description)/robots/parts/lidar_base/lidar_base.urdf.xacro"/>
   <xacro:include filename="$(find fws_robot_description)/robots/parts/lidar_head/lidar_head.urdf.xacro"/>
+  <xacro:include filename="$(find fws_robot_description)/robots/parts/imu/imu.urdf.xacro"/>
   <xacro:property name="M_PI" value="3.14159274"/>
   <material name="gray">
@@ -22,4 +23,8 @@
 	<origin xyz="0 0 0"/>
   </xacro:base_v0>
+  <!-- IMU -->
+  <xacro:imu_v0 parent="base_link">
+    <origin xyz="0 0 0.017"/>
+  </xacro:imu_v0>
   <!-- lidar_base -->
   <xacro:lidar_base_v0 parent="base_link">
@@ -75,4 +80,6 @@
   <!-- Base -->
   <xacro:base_gazebo_v0/>
+  <!-- IMU -->
+  <xacro:imu_gazebo_v0/>
   <!-- lidar base -->
   <xacro:lidar_base_gazebo_v0/>
