Commit message: added slam + nav2

File: racademy_ws/src/racademy_description/urdf/racademy.gazebo.xacro (robot description, xacro)
@@ -9,4 +9,23 @@
   <gazebo reference="camera_link">
     <material>Gazebo/Black</material>
+    <sensor name="camera_sensor" type="camera">
+      <always_on>true</always_on>
+      <visualize>true</visualize>
+      <update_rate>30</update_rate>
+      <topic>camera</topic>
+      <gz_frame_id>camera_optical_frame</gz_frame_id>
+      <camera>
+        <horizontal_fov>1.3962634</horizontal_fov>
+        <image>
+          <width>640</width>
+          <height>480</height>
+          <format>R8G8B8</format>
+        </image>
+        <clip>
+          <near>0.02</near>
+          <far>300</far>
+        </clip>
+      </camera>
+    </sensor>
   </gazebo>
   <gazebo reference="left_wheel_link">

File: racademy_ws/src/racademy_description/urdf/racademy.urdf.xacro (robot description, xacro)
@@ -168,3 +168,10 @@
     <origin xyz="0.08192 0.0 0.06161" rpy="0 0.1 0"/>
   </joint>
+  <!--  F.  Camera optical frame (Z-forward, X-right, Y-down convention for vision) -->
+  <link name="camera_optical_frame"/>
+  <joint name="camera_optical_joint" type="fixed">
+    <parent link="camera_link"/>
+    <child link="camera_optical_frame"/>
+    <origin xyz="0 0 0" rpy="-1.5707963 0 -1.5707963"/>
+  </joint>
 </robot>
